File: Sensorsboard.sch (EAGLE design)
At the start: 14 parts, among them U1 3.3v

Commit message: stuff
Parts:
- R1: value (none) -> 1k
Changed lines of the file:
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@@
 <part name="GND2" library="simple-shiled" library_urn="urn:adsk.eagle:library:80055" deviceset="GND" device=""/>
 <part name="D1" library="simple-shiled" library_urn="urn:adsk.eagle:library:80055" deviceset="LED-BLUE" device="0805" package3d_urn="urn:adsk.eagle:package:378040/2" value="POWER LED"/>
-<part name="R1" library="simple-shiled" library_urn="urn:adsk.eagle:library:80055" deviceset="RESISTOR" device="0805" package3d_urn="urn:adsk.eagle:package:103226/5" value=" "/>
+<part name="R1" library="simple-shiled" library_urn="urn:adsk.eagle:library:80055" deviceset="RESISTOR" device="0805" package3d_urn="urn:adsk.eagle:package:103226/5" value="1k"/>
 <part name="C1" library="simple-shiled" library_urn="urn:adsk.eagle:library:80055" deviceset="C-US" device="C1206K" package3d_urn="urn:adsk.eagle:package:878060/2"/>
 <part name="JP2" library="simple-shiled" library_urn="urn:adsk.eagle:library:80055" deviceset="PINHD-1X3" device="" package3d_urn="urn:adsk.eagle:package:80076/4"/>
